Commit message: fix: robot_foot_print origin

File: my_robot/urdf/my_robot.xacro (robot description, xacro)
@@ -5,5 +5,5 @@
   <link name="robot_footprint"></link>
   <joint name="robot_footprint_joint" type="fixed">
-    <origin xyz="0 0 0" rpy="0 0 0" />
+    <origin xyz="0 0 0.08" rpy="0 0 0" />
     <parent link="robot_footprint"/>
     <child link="chassis" />
